File: vesx/vesx.kicad_pcb (KiCad board)
At the start: 4 copper layers, 100 x 40 mm, 180 parts, among them J1 TYPE-C-31-M-12, J2 Conn_01x05, J3 Conn_01x06, J4 Conn_01x03, J5 Conn_01x04, J6 STLINK, J7 Conn_01x04, J8 CAN, U1 Opamp_Quad, U2 LM1117DT-3.3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

Commit message: fixed
Parts:
- moved J5 0.10 mm to (255.7, 32.6)
Connections:
- C11 pad 1: /MCU/VOLTAGE{PHASE} -> PA0
- C12 pad 1: /MCU/VOLTAGE{PHASE} -> PA1
- C13 pad 1: /MCU/VOLTAGE{PHASE} -> PA2
- R11 pad 1: /MCU/VOLTAGE{PHASE} -> PA2
- R22 pad 2: /MCU/VOLTAGE{PHASE} -> PA2
- R4 pad 1: /MCU/VOLTAGE{PHASE} -> PA0
- R6 pad 2: /MCU/VOLTAGE{PHASE} -> PA0
- R8 pad 1: /MCU/VOLTAGE{PHASE} -> PA1
- R9 pad 2: /MCU/VOLTAGE{PHASE} -> PA1
Routing:
- net PA2: track 3.60 -> 45.0 mm, vias 0 -> 2
- net PA0: track 3.31 -> 30.2 mm, vias 0 -> 2
- net PA1: track 3.39 -> 21.1 mm, vias 0 -> 2
- net GND: track 329.6 -> 315.5 mm, vias 332 -> 331
- net /MCU/VOLTAGE{PHASE}: track 11.5 -> 0.00 mm
- net Net-(U5-LVG): track 14.1 -> 2.69 mm

Commit message: Production
Parts:
- removed C51, C52: 4.7uF, Capacitor_SMD:C_0402_1005Metric
- added C28: 4.7uF, Capacitor_SMD:C_0603_1608Metric, F.Cu at (227.1, 44.5)
- added CX31: 470uF, CCC_ESC_Custom_parts:CAP_Polaryzed, F.Cu at (0.25, 0.25)
- added CX32: 470uF, CCC_ESC_Custom_parts:CAP_Polaryzed, F.Cu at (4.56, 0.25)
- added CX33: 470nF, Capacitor_SMD:C_1210_3225Metric, F.Cu at (2.33, 18.9)
- added CX34: 470uF, CCC_ESC_Custom_parts:CAP_Polaryzed, F.Cu at (8.87, 0.25)
- added CX35: 470nF, Capacitor_SMD:C_1210_3225Metric, F.Cu at (2.33, 23.2)
- added CX36: 470nF, Capacitor_SMD:C_1210_3225Metric, F.Cu at (2.33, 27.4)
- added CX37: 470uF, CCC_ESC_Custom_parts:CAP_Polaryzed, F.Cu at (13.2, 0.25)
- added CX38: 470nF, Capacitor_SMD:C_1210_3225Metric, F.Cu at (7.97, 18.9)
- added CX39: 470uF, CCC_ESC_Custom_parts:CAP_Polaryzed, F.Cu at (17.5, 0.25)
- added CX40: 470nF, Capacitor_SMD:C_1210_3225Metric, F.Cu at (7.97, 23.2)
- added CX41: 470uF, CCC_ESC_Custom_parts:CAP_Polaryzed, F.Cu at (21.8, 0.25)
- added CX42: 470nF, Capacitor_SMD:C_1210_3225Metric, F.Cu at (7.97, 27.4)
- added CX43: 470nF, Capacitor_SMD:C_1210_3225Metric, F.Cu at (13.6, 18.9)
- added CX44: 470uF, CCC_ESC_Custom_parts:CAP_Polaryzed, F.Cu at (26.1, 0.25)
- added CX45: 470nF, Capacitor_SMD:C_1210_3225Metric, F.Cu at (13.6, 23.2)
- added CX46: 470uF, CCC_ESC_Custom_parts:CAP_Polaryzed, F.Cu at (30.4, 0.25)
- added CX47: 470nF, Capacitor_SMD:C_1210_3225Metric, F.Cu at (13.6, 27.4)
- added CX48: 470nF, Capacitor_SMD:C_1210_3225Metric, F.Cu at (19.3, 18.9)
- added CX49: 470nF, Capacitor_SMD:C_1210_3225Metric, F.Cu at (19.3, 23.2)
- added CX51: 470nF, Capacitor_SMD:C_1210_3225Metric, F.Cu at (19.3, 27.4)
- C3: value 4u7 -> 4.7uF; footprint Capacitor_SMD:C_0402_1005Metric -> Capacitor_SMD:C_0603_1608Metric
- C4, C7: value 100n -> 100nf; footprint Capacitor_SMD:C_0402_1005Metric -> Capacitor_SMD:C_0603_1608Metric
- C41, C42, C47, C49, C50: footprint Capacitor_SMD:C_0402_1005Metric -> Capacitor_SMD:C_0603_1608Metric
- R34, R35, R36, R7: footprint Resistor_SMD:R_0402_1005Metric -> Resistor_SMD:R_0603_1608Metric
- moved C3 33.0 mm to (225.8, 44.5), turned to 90 degrees
- moved C7 1.67 mm to (193.1, 51.0)
- moved L1 1.28 mm to (225.5, 49.2)
- moved R34 1.24 mm to (181.0, 50.9)
- moved C42 1.14 mm to (192.7, 43.5)
- moved C49 1.00 mm to (223.2, 44.5)
- moved D6 1.00 mm to (179.6, 50.3)
- moved R15 0.95 mm to (230.9, 43.7)
- moved C41 0.85 mm to (192.8, 48.7)
- moved C4 0.81 mm to (191.6, 51.0)
- moved Y2 0.74 mm to (192.7, 46.1)
- moved D8 0.60 mm to (173.2, 50.3)
- moved C50 0.51 mm to (224.5, 44.5)
- moved C48 0.41 mm to (228.5, 44.4)
- moved R35 0.40 mm to (177.8, 50.9)
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Connections:
- C11 pad 1: PA0 -> /MCU/VOLTAGE{PHASE}
- C12 pad 1: PA1 -> /MCU/VOLTAGE{PHASE}
- C13 pad 1: PA2 -> /MCU/VOLTAGE{PHASE}
- C3 pad 1: +3V3 -> V12V
- C39 pad 1: CURRENT_A -> CURRENT_B
- C46 pad 1: CURRENT_C -> CURRENT_B
- D10 pad 2: CURRENT_C -> CURRENT_B
- D5 pad 2: CURRENT_A -> CURRENT_B
- R11 pad 1: PA2 -> /MCU/VOLTAGE{PHASE}
- R22 pad 2: PA2 -> /MCU/VOLTAGE{PHASE}
- R4 pad 1: PA0 -> /MCU/VOLTAGE{PHASE}
- R52 pad 2: CURRENT_A -> CURRENT_B
- R6 pad 2: PA0 -> /MCU/VOLTAGE{PHASE}
- R63 pad 2: CURRENT_C -> CURRENT_B
- R8 pad 1: PA1 -> /MCU/VOLTAGE{PHASE}
- R9 pad 2: PA1 -> /MCU/VOLTAGE{PHASE}
Routing:
- net GND: track 315.5 -> 290.7 mm, vias 331 -> 326
- net Net-(U5-LVG): track 2.69 -> 13.6 mm
- net +3V3: track 382.4 -> 376.6 mm, vias 36 -> 31
- net V12V: track 161.5 -> 158.4 mm, vias 11 -> 8
- net Net-(U3-FB): track 3.70 -> 5.14 mm
- net LED_R: track 13.3 -> 14.7 mm
- net Net-(U7-PH1): track 10.2 -> 11.1 mm

Commit message: prob final
Parts:
- removed CX31, CX32, CX34, CX37, CX39, CX41, CX44, CX46: 470uF, CCC_ESC_Custom_parts:CAP_Polaryzed
- removed CX33, CX35, CX36, CX38, CX40, CX42, CX48, CX49: 470nF, Capacitor_SMD:C_1210_3225Metric
- CX43, CX45, CX47, CX51: moved to B.Cu
- PHASE_A: value MountingHole_3.5mm_Pad -> MountingHole_3.0mm_Pad; footprint (none) -> MountingHole:MountingHole_3.2mm_M3_DIN965_Pad_TopBottom
- PHASE_B: footprint (none) -> MountingHole:MountingHole_3.2mm_M3_DIN965_Pad_TopBottom
- PHASE_C: value MountingHole_3.5mm_Pad -> MountingHole_3.2mm_M3_DIN965_Pad_TopBottom; footprint MountingHole:MountingHole_3.5mm_Pad -> MountingHole:MountingHole_3.2mm_M3_DIN965_Pad_TopBottom
- moved CX43 197.9 mm to (211.5, 24.0), turned to 180 degrees
- moved CX45 171.9 mm to (185.5, 24.0), turned to 180 degrees
- moved CX47 151.8 mm to (165.0, 16.0)
- moved CX51 141.3 mm to (160.5, 24.5), turned to 180 degrees
Connections:
- C11 pad 1: /MCU/VOLTAGE{PHASE} -> PA0
- C12 pad 1: /MCU/VOLTAGE{PHASE} -> PA1
- C13 pad 1: /MCU/VOLTAGE{PHASE} -> PA2
- C39 pad 1: CURRENT_B -> CURRENT_A
- C46 pad 1: CURRENT_B -> CURRENT_C
- D10 pad 2: CURRENT_B -> CURRENT_C
- D5 pad 2: CURRENT_B -> CURRENT_A
- R11 pad 1: /MCU/VOLTAGE{PHASE} -> PA2
- R2 pad 2: PB10 -> DUAL2_RX
- R22 pad 2: /MCU/VOLTAGE{PHASE} -> PA2
- R3 pad 1: PB10 -> DUAL1_TX
- R4 pad 1: /MCU/VOLTAGE{PHASE} -> PA0
- R52 pad 2: CURRENT_B -> CURRENT_A
- R6 pad 2: /MCU/VOLTAGE{PHASE} -> PA0
- R63 pad 2: CURRENT_B -> CURRENT_C
- R8 pad 1: /MCU/VOLTAGE{PHASE} -> PA1
- R9 pad 2: /MCU/VOLTAGE{PHASE} -> PA1
- U7 pad 29: PB10 -> DUAL1_TX
- U7 pad 30: PB10 -> DUAL2_RX
Routing:
- net VBAT: track 197.0 -> 204.9 mm
- net GND: track 290.7 -> 291.1 mm, vias 326 -> 358
- net CL: track 46.3 -> 46.6 mm, vias 2 -> 3
