File: vesx/PSense.kicad_sch (KiCad schematic)
At the start: 97 parts, among them U1 Opamp_Quad, U5 L6498DTR, U6 L6498DTR, U8 L6498DTR

Commit message: aaaaaaaaaaaaaaaaaaaaaaaaaaaaaaaaaaaaaaaa
Parts:
- C11, C12, C13: LCSC C1671 -> C1671
- C14, C15, C20, C36: LCSC (none) -> C14663
- C17, C35, C37: LCSC (none) -> C96446
- C2: LCSC (none) -> C1525
- C38: value C_Small -> 10nF; LCSC (none) -> C57112
- C39, C40, C46: LCSC (none) -> C1588
- CX31, CX32, CX34, CX37, CX39, CX41, CX44, CX46: now not fitted
- D1, D2, D3: LCSC (none) -> C191023; now not fitted
- D10, D5, D9: LCSC (none) -> C191023
- R1: LCSC (none) -> C25118
- R23, R28, R38: LCSC (none) -> C22939
- R24, R26, R29, R31, R39, R41, R46: LCSC (none) -> C25804
- R25, R27, R30, R32, R40, R42: LCSC (none) -> C23214
- R43, R51, R54, R59: LCSC (none) -> C25803
- R44: LCSC (none) -> C31850
- R45: LCSC (none) -> C21190
- R47: LCSC (none) -> C22961
- R48: LCSC (none) -> C23182
- R49, R50, R55, R56, R60, R61: LCSC (none) -> C4190
- R52, R58, R63: LCSC (none) -> C22808
- R53, R57, R62: LCSC (none) -> C25819
- SH1, SH2, SH3: LCSC (none) -> C7178835
- U1: LCSC (none) -> C695777
- U5, U6, U8: LCSC (none) -> C500658

Commit message: Production
Parts:
- removed CX31, CX32, CX34, CX37, CX39, CX41, CX44, CX46: 470uF, CCC_ESC_Custom_parts:CAP_Polaryzed, symbol Device:C_Polarized
- removed CX33, CX35, CX36, CX38, CX40, CX42, CX43, CX45, CX47, CX48, CX49, CX51: 470nF, Capacitor_SMD:C_1210_3225Metric, symbol Device:C

Commit message: asdf
Parts:
- D1, D2, D3: LCSC C191023 -> C412437; now fitted
Changed lines of the file:
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@@
 		(in_bom yes)
 		(on_board yes)
-		(dnp yes)
+		(dnp no)
 		(fields_autoplaced yes)
 		(property "Reference" "D1"
@@
 			)
 		)
-		(property "LCSC" "C191023"
+		(property "LCSC" " C412437"
 			(at 195.58 21.59 0)
 			(effects
@@
 		(in_bom yes)
 		(on_board yes)
-		(dnp yes)
+		(dnp no)
 		(fields_autoplaced yes)
 		(property "Reference" "D2"
@@
 			)
 		)
-		(property "LCSC" "C191023"
+		(property "LCSC" " C412437"
 			(at 195.58 68.58 0)
 			(effects
@@
 		(in_bom yes)
 		(on_board yes)
-		(dnp yes)
+		(dnp no)
 		(fields_autoplaced yes)
 		(property "Reference" "D3"
@@
 			)
 		)
-		(property "LCSC" "C191023"
+		(property "LCSC" " C412437"
 			(at 195.58 118.11 0)
 			(effects

Commit message: prob final
Parts:
- QA1, QA2, QA3, QA4, QA5, QA6: now not fitted
