File: vesx/vesx.kicad_sch (KiCad schematic)
At the start: 80 parts, among them J1 TYPE-C-31-M-12, J2 Conn_01x05, J3 Conn_01x06, J4 Conn_01x03, J5 Conn_01x04, J7 Conn_01x04, U3 LM5164DDA, U4 TO220_replacement_module

Commit message: aaaaaaaaaaaaaaaaaaaaaaaaaaaaaaaaaaaaaaaa
Parts:
- removed CX1, CX2, CX3, CX4, CX5, CX6, CX7, CX8: 470uF, CCC_ESC_Custom_parts:CAP_Polaryzed, symbol Device:C_Polarized
- removed CX10, CX11, CX12, CX13, CX14, CX25, CX26, CX27, CX28, CX29, CX30: 470nF, Capacitor_SMD:C_1210_3225Metric, symbol Device:C
- C21, C22, C23: LCSC (none) -> C1588
- C24: value 100nF -> 1nF; LCSC (none) -> C1588
- C26: LCSC (none) -> C6119850
- C27: now not fitted
- C30, C31: LCSC (none) -> C15849
- C43: footprint Capacitor_SMD:C_1210_3225Metric -> Capacitor_SMD:C_0603_1608Metric; LCSC (none) -> C96446
- C47: LCSC (none) -> C385029
- C48: LCSC (none) -> C343868
- C49: footprint Capacitor_SMD:C_0402_1005Metric -> Capacitor_SMD:C_0603_1608Metric; LCSC (none) -> C14663
- C50, C51, C52: LCSC (none) -> C23733
- D11: LCSC (none) -> C2903858
- D12: LCSC (none) -> C508230
- L1: footprint Inductor_SMD:L_Abracon_ASPI-4030S -> Inductor_SMD:L_TracoPower_TCK-047_5.2x5.8mm; LCSC (none) -> C5362907
- R10, RN1, RN2: LCSC (none) -> C25804
- R15: LCSC (none) -> C2828635
- R5: LCSC (none) -> C3016359
- R7: LCSC (none) -> C3015903
- TH1: LCSC (none) -> C167506; now not fitted
- U3: LCSC (none) -> C477928

Commit message: Production
Parts:
- removed C51, C52: 4.7uF, Capacitor_SMD:C_0402_1005Metric, symbol Device:C_Small
- removed CX15, CX16, CX17, CX18, CX19, CX20, CX21, CX22: 470nF, Capacitor_SMD:C_1210_3225Metric, symbol Device:C
- added C28, C3: 4.7uF, Capacitor_SMD:C_0603_1608Metric, symbol Device:C_Small
- C47: footprint Capacitor_SMD:C_0402_1005Metric -> Capacitor_SMD:C_0603_1608Metric; LCSC C385029 -> C113804
- C50: footprint Capacitor_SMD:C_0402_1005Metric -> Capacitor_SMD:C_0603_1608Metric; LCSC C23733 -> C237615
- R15: footprint Resistor_SMD:R_0402_1005Metric -> Resistor_SMD:R_0603_1608Metric
- R7: footprint Resistor_SMD:R_0402_1005Metric -> Resistor_SMD:R_0603_1608Metric; LCSC C3015903 -> C269687
Connections:
- net +12V: now also C28.1, C3.1
- net GND: now also C28.2, C3.2

Commit message: asdf
Parts:
- J2, J3, J4, J5, J7: now not fitted
- RN1, RN2: LCSC C25804 -> C20624287
- TH1: now fitted
Other:
- moved on the sheet: C27
Changed lines of the file:
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@@
 	)
 	(junction
-		(at 107.95 226.06)
-		(diameter 0)
-		(color 0 0 0 0)
-	)
-	(junction
 		(at 179.07 138.43)
 		(diameter 0)
@@
 	)
 	(junction
-		(at 43.18 259.08)
+		(at 106.68 246.38)
 		(diameter 0)
 		(color 0 0 0 0)
 	)
 	(junction
-		(at 346.71 233.68)
+		(at 43.18 259.08)
 		(diameter 0)
 		(color 0 0 0 0)
 	)
 	(junction
-		(at 107.95 246.38)
+		(at 346.71 233.68)
 		(diameter 0)
 		(color 0 0 0 0)
@@
 	)
 	(junction
+		(at 106.68 226.06)
+		(diameter 0)
+		(color 0 0 0 0)
+	)
+	(junction
 		(at 261.62 119.38)
 		(diameter 0)
@@
 	(wire
 		(pts
-			(xy 107.95 238.76) (xy 107.95 246.38)
+			(xy 106.68 240.03) (xy 106.68 246.38)
 		)
 		(stroke
@@
 	(wire
 		(pts
+			(xy 106.68 246.38) (xy 111.76 246.38)
+		)
+		(stroke
+			(width 0)
+			(type default)
+		)
+	)
+	(wire
+		(pts
 			(xy 285.75 172.72) (xy 295.91 172.72)
 		)
@@
 	(wire
 		(pts
-			(xy 100.33 246.38) (xy 107.95 246.38)
+			(xy 100.33 246.38) (xy 106.68 246.38)
 		)
 		(stroke
@@
 	(wire
 		(pts
-			(xy 107.95 226.06) (xy 107.95 231.14)
+			(xy 106.68 226.06) (xy 106.68 232.41)
 		)
 		(stroke
@@
 	(wire
 		(pts
-			(xy 100.33 226.06) (xy 107.95 226.06)
+			(xy 100.33 226.06) (xy 106.68 226.06)
 		)
 		(stroke
@@
 	(wire
 		(pts
-			(xy 107.95 246.38) (xy 111.76 246.38)
-		)
-		(stroke
-			(width 0)
-			(type default)
-		)
-	)
-	(wire
-		(pts
 			(xy 64.77 238.76) (xy 64.77 245.11)
 		)
@@
 	(wire
 		(pts
-			(xy 354.33 219.71) (xy 354.33 222.25)
+			(xy 106.68 226.06) (xy 111.76 226.06)
 		)
 		(stroke
@@
 	(wire
 		(pts
-			(xy 107.95 226.06) (xy 111.76 226.06)
+			(xy 354.33 219.71) (xy 354.33 222.25)
 		)
 		(stroke
@@
 		(in_bom yes)
 		(on_board yes)
-		(dnp yes)
+		(dnp no)
 		(fields_autoplaced yes)
 		(property "Reference" "TH1"
@@
 			)
 		)
-		(property "LCSC" " C25804"
+		(property "LCSC" "C20624287"
 			(at 38.1 105.41 0)
 			(effects
@@
 		(in_bom yes)
 		(on_board yes)
-		(dnp no)
+		(dnp yes)
 		(fields_autoplaced yes)
 		(property "Reference" "J2"
@@
 	(symbol
 		(lib_id "Device:C_Polarized")
-		(at 107.95 234.95 0)
+		(at 106.68 236.22 0)
 		(unit 1)
 		(exclude_from_sim no)
@@
 		(fields_autoplaced yes)
 		(property "Reference" "C27"
-			(at 111.76 232.7909 0)
+			(at 110.49 234.0609 0)
 			(effects
 				(font
@@
 		)
 		(property "Value" "C_Polarized"
-			(at 111.76 235.3309 0)
+			(at 110.49 236.6009 0)
 			(effects
 				(font
@@
 		)
 		(property "Footprint" "Capacitor_THT:CP_Radial_D8.0mm_P3.50mm"
-			(at 108.9152 238.76 0)
+			(at 107.6452 240.03 0)
 			(effects
 				(font
@@
 		)
 		(property "Datasheet" "~"
-			(at 107.95 234.95 0)
+			(at 106.68 236.22 0)
 			(effects
 				(font
@@
 		)
 		(property "Description" "Polarized capacitor"
-			(at 107.95 234.95 0)
+			(at 106.68 236.22 0)
 			(effects
 				(font
@@
 		(in_bom yes)
 		(on_board yes)
-		(dnp no)
+		(dnp yes)
 		(property "Reference" "J7"
 			(at 144.526 213.36 90)
@@
 		(in_bom yes)
 		(on_board yes)
-		(dnp no)
+		(dnp yes)
 		(property "Reference" "J3"
 			(at 27.94 111.76 0)
@@
 		(in_bom yes)
 		(on_board yes)
-		(dnp no)
+		(dnp yes)
 		(fields_autoplaced yes)
 		(property "Reference" "J5"
@@
 		(in_bom yes)
 		(on_board yes)
-		(dnp no)
+		(dnp yes)
 		(property "Reference" "J4"
 			(at 119.38 217.1699 90)
@@
 			)
 		)
-		(property "LCSC" " C25804"
+		(property "LCSC" "C20624287"
 			(at 50.8 123.19 0)
 			(effects

Commit message: prob final
Parts:
- U4: now not fitted
Other:
- moved on the sheet: CX23, CX24
